Commit message: add hand

File: robot/fr3.urdf (robot description, URDF)
Before this commit: robot fr3, 10 links, 9 joints
Links:
- added link fr3_hand, mass 0.6544; collision box size=0.04 0.201 0.075; visual mesh filename=package://mujoco_ros_sim/mujoco_menagerie/franka_fr3_torque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
- added link fr3_hand_tcp
- added link fr3_leftfinger, mass 0.0291; visual mesh filename=package://mujoco_ros_sim/mujoco_menagerie/franka_fr3_torque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
- added link fr3_rightfinger, mass 0.0291; visual mesh filename=package://mujoco_ros_sim/mujoco_menagerie/franka_fr3_torque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
Joints:
- added joint fr3_finger_joint1: type fixed, parent fr3_hand, child fr3_leftfinger, origin xyz=0 0 0.0584 rpy=0 0 0
- added joint fr3_finger_joint2: type fixed, parent fr3_hand, child fr3_rightfinger, origin xyz=0 0 0.0584 rpy=0 0 3.141592653589793
- added joint fr3_hand_joint: type fixed, parent fr3_link8, child fr3_hand, origin xyz=0 0 0 rpy=0 0 -0.7853981633974483
- added joint fr3_hand_tcp_joint: type fixed, parent fr3_hand, child fr3_hand_tcp, origin xyz=0 0 0.1034 rpy=0 0 0

Commit message: add franka hand

File: robot/fr3.urdf (robot description, URDF)
Before this commit: robot fr3, 14 links, 13 joints
Links:
- link fr3_hand: mass 0.6544 -> 0.73
- link fr3_leftfinger: mass 0.0291 -> 0.015
- link fr3_rightfinger: mass 0.0291 -> 0.015

File: robot/fr3_husky.urdf (robot description, URDF)
Before this commit: robot fr3_husky, 24 links, 23 joints
Links:
- added link fr3_hand, mass 0.73; collision box size=0.04 0.201 0.075; visual mesh filename=package://mujoco_ros_sim/mujoco_menagerie/franka_fr3_torque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
- added link fr3_hand_tcp
- added link fr3_leftfinger, mass 0.015; visual mesh filename=package://mujoco_ros_sim/mujoco_menagerie/franka_fr3_torque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
- added link fr3_rightfinger, mass 0.015; visual mesh filename=package://mujoco_ros_sim/mujoco_menagerie/franka_fr3_torque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
- link left_wheel: geometry 
- link right_wheel: geometry 
Joints:
- added joint fr3_finger_joint1: type fixed, parent fr3_hand, child fr3_leftfinger, origin xyz=0 0 0.0584 rpy=0 0 0
- added joint fr3_finger_joint2: type fixed, parent fr3_hand, child fr3_rightfinger, origin xyz=0 0 0.0584 rpy=0 0 3.141592653589793
- added joint fr3_hand_joint: type fixed, parent fr3_link8, child fr3_hand, origin xyz=0 0 0 rpy=0 0 -0.7853981633974483
- added joint fr3_hand_tcp_joint: type fixed, parent fr3_hand, child fr3_hand_tcp, origin xyz=0 0 0.1034 rpy=0 0 0

File: robot/fr3_pcv.urdf (robot description, URDF)
Before this commit: robot fr3_pcv, 23 links, 22 joints
Links:
- added link fr3_hand, mass 0.73; collision box size=0.04 0.201 0.075; visual mesh filename=package://mujoco_ros_sim/mujoco_menagerie/franka_fr3_torque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
- added link fr3_hand_tcp
- added link fr3_leftfinger, mass 0.015; visual mesh filename=package://mujoco_ros_sim/mujoco_menagerie/franka_fr3_torque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
- added link fr3_rightfinger, mass 0.015; visual mesh filename=package://mujoco_ros_sim/mujoco_menagerie/franka_fr3_torque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
Joints:
- added joint fr3_finger_joint1: type fixed, parent fr3_hand, child fr3_leftfinger, origin xyz=0 0 0.0584 rpy=0 0 0
- added joint fr3_finger_joint2: type fixed, parent fr3_hand, child fr3_rightfinger, origin xyz=0 0 0.0584 rpy=0 0 3.141592653589793
- added joint fr3_hand_joint: type fixed, parent fr3_link8, child fr3_hand, origin xyz=0 0 0 rpy=0 0 -0.7853981633974483
- added joint fr3_hand_tcp_joint: type fixed, parent fr3_hand, child fr3_hand_tcp, origin xyz=0 0 0.1034 rpy=0 0 0

File: robot/fr3_xls.urdf (robot description, URDF)
Before this commit: robot fr3_xls, 25 links, 24 joints
Links:
- added link fr3_hand, mass 0.73; collision box size=0.04 0.201 0.075; visual mesh filename=package://mujoco_ros_sim/mujoco_menagerie/franka_fr3_torque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
- added link fr3_hand_tcp
- added link fr3_leftfinger, mass 0.015; visual mesh filename=package://mujoco_ros_sim/mujoco_menagerie/franka_fr3_torque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
- added link fr3_rightfinger, mass 0.015; visual mesh filename=package://mujoco_ros_sim/mujoco_menagerie/franka_fr3_torque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
Joints:
- added joint fr3_finger_joint1: type fixed, parent fr3_hand, child fr3_leftfinger, origin xyz=0 0 0.0584 rpy=0 0 0
- added joint fr3_finger_joint2: type fixed, parent fr3_hand, child fr3_rightfinger, origin xyz=0 0 0.0584 rpy=0 0 3.141592653589793
- added joint fr3_hand_joint: type fixed, parent fr3_link8, child fr3_hand, origin xyz=0 0 0 rpy=0 0 -0.7853981633974483
- added joint fr3_hand_tcp_joint: type fixed, parent fr3_hand, child fr3_hand_tcp, origin xyz=0 0 0.1034 rpy=0 0 0
