Commit message: add fr3_husky

File: robot/fr3_husky.urdf (robot description, URDF)
Before this commit: robot fr3_husky, 24 links, 23 joints
Links:
- link top_structure_link: mass None -> 36.436; geometry collision box size=0.25 0.35 0.01; collision box size=0.32 0.56 1.3
Joints:
- joint top_structure_joint: origin xyz=0 0 0 rpy=0 0 0 -> xyz=0 0 0.248 rpy=0 0 0

Commit message: add wheel collision model

File: robot/fr3_husky.urdf (robot description, URDF)
Before this commit: robot fr3_husky, 28 links, 27 joints
Links:
- link front_left_wheel: geometry collision cylinder length=0.1143 radius=0.1651; visual mesh filename=package://mujoco_ros_sim/mujoco_menagerie/fr3_husky/assets/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
- link front_right_wheel: geometry collision cylinder length=0.1143 radius=0.1651; visual mesh filename=package://mujoco_ros_sim/mujoco_menagerie/fr3_husky/assets/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
- link rear_left_wheel: geometry collision cylinder length=0.1143 radius=0.1651; visual mesh filename=package://mujoco_ros_sim/mujoco_menagerie/fr3_husky/assets/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
- link rear_right_wheel: geometry collision cylinder length=0.1143 radius=0.1651; visual mesh filename=package://mujoco_ros_sim/mujoco_menagerie/fr3_husky/assets/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

Commit message: fix fr3_husky urdf

File: robot/fr3_husky.urdf (robot description, URDF)
Before this commit: robot fr3_husky, 28 links, 27 joints
Joints:
- joint fr3_base_joint: origin xyz=0.36 0.0 0.256 rpy=0 0 0 -> xyz=0.36 0.0 0.27 rpy=0 0 0
