Commit message: fix typo

File: robot/dual_fr3_husky.urdf (robot description, URDF)
Before this commit: robot dual_dual_fr3_husky, 41 links, 40 joints
Joints:
- joint r_fr3_base_joint: origin xyz=0.345 -0.215 0.26 rpy=0 0 -0.523598776 -> xyz=0.345 0.215 0.26 rpy=0 0 0.523598776

Commit message: fix top structure

File: robot/dual_fr3_husky.urdf (robot description, URDF)
Before this commit: robot dual_dual_fr3_husky, 41 links, 40 joints
Links:
- link top_structure_link: geometry collision box size=0.32 0.56 1.3; collision box size=0.85 0.65 0.012

Commit message: fix name

File: robot/dual_fr3_husky.urdf (robot description, URDF)
Before this commit: robot dual_dual_fr3_husky, 41 links, 40 joints
Links:
- removed link l_fr3_hand
- removed link l_fr3_hand_tcp
- removed link l_fr3_leftfinger
- removed link l_fr3_link0
- removed link l_fr3_link1
- removed link l_fr3_link2
- removed link l_fr3_link3
- removed link l_fr3_link4
- removed link l_fr3_link5
- removed link l_fr3_link6
- removed link l_fr3_link7
- removed link l_fr3_link8
- removed link l_fr3_rightfinger
- removed link r_fr3_hand
- removed link r_fr3_hand_tcp
- removed link r_fr3_leftfinger
- removed link r_fr3_link0
- removed link r_fr3_link1
- removed link r_fr3_link2
- removed link r_fr3_link3
- removed link r_fr3_link4
- removed link r_fr3_link5
- removed link r_fr3_link6
- removed link r_fr3_link7
- removed link r_fr3_link8
- removed link r_fr3_rightfinger
- added link fr3_l_hand, mass 0.73; collision box size=0.04 0.201 0.075; visual mesh filename=package://mujoco_ros_sim/mujoco_menagerie/dual_fr3_husky/as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
- added link fr3_l_hand_tcp
- added link fr3_l_leftfinger, mass 0.015; visual mesh filename=package://mujoco_ros_sim/mujoco_menagerie/dual_fr3_husky/as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
- added link fr3_l_link0, mass 2.3966; collision cylinder length=0.03 radius=0.07; collision cylinder length=0.06 radius=0.07
- added link fr3_l_link1, mass 2.9274653454; collision cylinder length=0.12 radius=0.065; collision cylinder length=0.2830 radius=0.07
- added link fr3_l_link2, mass 2.9355370338; collision cylinder length=0.12 radius=0.065; collision cylinder length=0.12 radius=0.07
- added link fr3_l_link3, mass 2.2449013699; collision cylinder length=0.15 radius=0.07; collision sphere radius=0.07
- added link fr3_l_link4, mass 2.6155955791; collision cylinder length=0.02 radius=0.07; collision cylinder length=0.02 radius=0.07
- added link fr3_l_link5, mass 2.3271207594; collision cylinder length=0.1 radius=0.07; collision cylinder length=0.17 radius=0.045
- added link fr3_l_link6, mass 1.8170376524; collision cylinder length=0.07 radius=0.07; collision cylinder length=0.08 radius=0.07
- added link fr3_l_link7, mass 0.6271432862; collision box size=0.071 0.071 0.041; collision cylinder length=0.05 radius=0.051
- added link fr3_l_link8
- added link fr3_l_rightfinger, mass 0.015; visual mesh filename=package://mujoco_ros_sim/mujoco_menagerie/dual_fr3_husky/as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
- added link fr3_r_hand, mass 0.73; collision box size=0.04 0.201 0.075; visual mesh filename=package://mujoco_ros_sim/mujoco_menagerie/dual_fr3_husky/as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
- added link fr3_r_hand_tcp
- added link fr3_r_leftfinger, mass 0.015; visual mesh filename=package://mujoco_ros_sim/mujoco_menagerie/dual_fr3_husky/as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
- added link fr3_r_link0, mass 2.3966; collision cylinder length=0.03 radius=0.07; collision cylinder length=0.06 radius=0.07
- added link fr3_r_link1, mass 2.9274653454; collision cylinder length=0.12 radius=0.065; collision cylinder length=0.2830 radius=0.07
- added link fr3_r_link2, mass 2.9355370338; collision cylinder length=0.12 radius=0.065; collision cylinder length=0.12 radius=0.07
- added link fr3_r_link3, mass 2.2449013699; collision cylinder length=0.15 radius=0.07; collision sphere radius=0.07
- added link fr3_r_link4, mass 2.6155955791; collision cylinder length=0.02 radius=0.07; collision cylinder length=0.02 radius=0.07
- added link fr3_r_link5, mass 2.3271207594; collision cylinder length=0.1 radius=0.07; collision cylinder length=0.17 radius=0.045
- added link fr3_r_link6, mass 1.8170376524; collision cylinder length=0.07 radius=0.07; collision cylinder length=0.08 radius=0.07
- added link fr3_r_link7, mass 0.6271432862; collision box size=0.071 0.071 0.041; collision cylinder length=0.05 radius=0.051
- added link fr3_r_link8
- added link fr3_r_rightfinger, mass 0.015; visual mesh filename=package://mujoco_ros_sim/mujoco_menagerie/dual_fr3_husky/as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
Joints:
- removed joint l_fr3_base_joint
- removed joint l_fr3_finger_joint1
- removed joint l_fr3_finger_joint2
- removed joint l_fr3_hand_joint
- removed joint l_fr3_hand_tcp_joint
- removed joint l_fr3_joint1
- removed joint l_fr3_joint2
- removed joint l_fr3_joint3
- removed joint l_fr3_joint4
- removed joint l_fr3_joint5
- removed joint l_fr3_joint6
- removed joint l_fr3_joint7
- removed joint l_fr3_joint8
- removed joint r_fr3_base_joint
- removed joint r_fr3_finger_joint1
- removed joint r_fr3_finger_joint2
- removed joint r_fr3_hand_joint
- removed joint r_fr3_hand_tcp_joint
- removed joint r_fr3_joint1
- removed joint r_fr3_joint2
- removed joint r_fr3_joint3
- removed joint r_fr3_joint4
- removed joint r_fr3_joint5
- removed joint r_fr3_joint6
- removed joint r_fr3_joint7
- removed joint r_fr3_joint8
- added joint fr3_l_base_joint: type fixed, parent base_link, child fr3_l_link0, origin xyz=0.345 0.215 0.26 rpy=0 0 0.523598776
- added joint fr3_l_finger_joint1: type fixed, parent fr3_l_hand, child fr3_l_leftfinger, origin xyz=0 0 0.0584 rpy=0 0 0
- added joint fr3_l_finger_joint2: type fixed, parent fr3_l_hand, child fr3_l_rightfinger, origin xyz=0 0 0.0584 rpy=0 0 3.141592653589793
- added joint fr3_l_hand_joint: type fixed, parent fr3_l_link8, child fr3_l_hand, origin xyz=0 0 0 rpy=0 0 -0.7853981633974483
- added joint fr3_l_hand_tcp_joint: type fixed, parent fr3_l_hand, child fr3_l_hand_tcp, origin xyz=0 0 0.1034 rpy=0 0 0
- added joint fr3_l_joint1: type revolute, parent fr3_l_link0, child fr3_l_link1, origin xyz=0 0 0.333 rpy=0 0 0, axis 0 0 1, limit lower=-2.7437 upper=2.7437 effort=87.0 velocity=2.62
- added joint fr3_l_joint2: type revolute, parent fr3_l_link1, child fr3_l_link2, origin xyz=0 0 0 rpy=-1.570796326794897 0 0, axis 0 0 1, limit lower=-1.7837 upper=1.7837 effort=87.0 velocity=2.62
- added joint fr3_l_joint3: type revolute, parent fr3_l_link2, child fr3_l_link3, origin xyz=0 -0.316 0 rpy=1.570796326794897 0 0, axis 0 0 1, limit lower=-2.9007 upper=2.9007 effort=87.0 velocity=2.62
- added joint fr3_l_joint4: type revolute, parent fr3_l_link3, child fr3_l_link4, origin xyz=0.0825 0 0 rpy=1.570796326794897 0 0, axis 0 0 1, limit lower=-3.0421 upper=-0.1518 effort=87.0 velocity=2.62
- added joint fr3_l_joint5: type revolute, parent fr3_l_link4, child fr3_l_link5, origin xyz=-0.0825 0.384 0 rpy=-1.570796326794897 0 0, axis 0 0 1, limit lower=-2.8065 upper=2.8065 effort=12.0 velocity=5.26
- added joint fr3_l_joint6: type revolute, parent fr3_l_link5, child fr3_l_link6, origin xyz=0 0 0 rpy=1.570796326794897 0 0, axis 0 0 1, limit lower=0.5445 upper=4.5169 effort=12.0 velocity=4.18
- added joint fr3_l_joint7: type revolute, parent fr3_l_link6, child fr3_l_link7, origin xyz=0.088 0 0 rpy=1.570796326794897 0 0, axis 0 0 1, limit lower=-3.0159 upper=3.0159 effort=12.0 velocity=5.26
- added joint fr3_l_joint8: type fixed, parent fr3_l_link7, child fr3_l_link8, origin xyz=0 0 0.107 rpy=0 0 0
- added joint fr3_r_base_joint: type fixed, parent base_link, child fr3_r_link0, origin xyz=0.345 -0.215 0.26 rpy=0 0 -0.523598776
- added joint fr3_r_finger_joint1: type fixed, parent fr3_r_hand, child fr3_r_leftfinger, origin xyz=0 0 0.0584 rpy=0 0 0
- added joint fr3_r_finger_joint2: type fixed, parent fr3_r_hand, child fr3_r_rightfinger, origin xyz=0 0 0.0584 rpy=0 0 3.141592653589793
- added joint fr3_r_hand_joint: type fixed, parent fr3_r_link8, child fr3_r_hand, origin xyz=0 0 0 rpy=0 0 -0.7853981633974483
- added joint fr3_r_hand_tcp_joint: type fixed, parent fr3_r_hand, child fr3_r_hand_tcp, origin xyz=0 0 0.1034 rpy=0 0 0
- added joint fr3_r_joint1: type revolute, parent fr3_r_link0, child fr3_r_link1, origin xyz=0 0 0.333 rpy=0 0 0, axis 0 0 1, limit lower=-2.7437 upper=2.7437 effort=87.0 velocity=2.62
- added joint fr3_r_joint2: type revolute, parent fr3_r_link1, child fr3_r_link2, origin xyz=0 0 0 rpy=-1.570796326794897 0 0, axis 0 0 1, limit lower=-1.7837 upper=1.7837 effort=87.0 velocity=2.62
- added joint fr3_r_joint3: type revolute, parent fr3_r_link2, child fr3_r_link3, origin xyz=0 -0.316 0 rpy=1.570796326794897 0 0, axis 0 0 1, limit lower=-2.9007 upper=2.9007 effort=87.0 velocity=2.62
- added joint fr3_r_joint4: type revolute, parent fr3_r_link3, child fr3_r_link4, origin xyz=0.0825 0 0 rpy=1.570796326794897 0 0, axis 0 0 1, limit lower=-3.0421 upper=-0.1518 effort=87.0 velocity=2.62
- added joint fr3_r_joint5: type revolute, parent fr3_r_link4, child fr3_r_link5, origin xyz=-0.0825 0.384 0 rpy=-1.570796326794897 0 0, axis 0 0 1, limit lower=-2.8065 upper=2.8065 effort=12.0 velocity=5.26
- added joint fr3_r_joint6: type revolute, parent fr3_r_link5, child fr3_r_link6, origin xyz=0 0 0 rpy=1.570796326794897 0 0, axis 0 0 1, limit lower=0.5445 upper=4.5169 effort=12.0 velocity=4.18
- added joint fr3_r_joint7: type revolute, parent fr3_r_link6, child fr3_r_link7, origin xyz=0.088 0 0 rpy=1.570796326794897 0 0, axis 0 0 1, limit lower=-3.0159 upper=3.0159 effort=12.0 velocity=5.26
- added joint fr3_r_joint8: type fixed, parent fr3_r_link7, child fr3_r_link8, origin xyz=0 0 0.107 rpy=0 0 0
